File: PuyoPuya/PuyoPuya.kicad_sch (KiCad schematic)
At the start: 17 parts, among them J1 Conn_01x10, J2 SWD, J3 USB4085-GF-A, SW1 SW_Push, U1 PY32F003W16S6TU

Commit message: Boarb
Parts:
- J1: value Conn_01x10 -> Conn_02x10; footprint Connector_PinSocket_2.54mm:PinSocket_1x10_P2.54mm_Vertical -> Connector_PinSocket_2.54mm:PinSocket_2x10_P2.54mm_Vertical; symbol Connector_Generic:Conn_01x10 -> Connector_Generic:Conn_02x10_Odd_Even
Connections:
- net SWCLK is gone; now on net SWDCLK: J2.4 (Pin_4)
- net GND: now also J1.14 (Pin_14), J1.16 (Pin_16), J1.18 (Pin_18), J1.20 (Pin_20), J3.B12 (GND)
- net PA1: now also J1.3 (Pin_3); no longer J1.2 (Pin_2)
- net PA12: now also J1.17 (Pin_17); no longer J1.9 (Pin_9)
- net PA13/SWDIO: now also J1.19 (Pin_19); no longer J1.10 (Pin_10)
- net PA2: now also J1.5 (Pin_5); no longer J1.3 (Pin_3)
- net PA3: now also J1.7 (Pin_7); no longer J1.4 (Pin_4)
- net PA4: now also J1.9 (Pin_9); no longer J1.5 (Pin_5)
- net PA5: now also J1.11 (Pin_11); no longer J1.6 (Pin_6)
- net PA6: now also J1.13 (Pin_13); no longer J1.7 (Pin_7)
- net PA7: now also J1.15 (Pin_15); no longer J1.8 (Pin_8)
- net PB0: now also J1.2 (Pin_2)
- net PB1: now also J1.4 (Pin_4)
- net VCC: now also J1.10 (Pin_10), J1.12 (Pin_12), J1.6 (Pin_6), J1.8 (Pin_8)
- no-connect marks 11 -> 10
Changed lines of the file:
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@@
 (kicad_sch (version 20230121) (generator eeschema)
   (paper "A4")
+  (junction (at 186.69 86.995) (diameter 0) (color 0 0 0 0)
+  )
+  (junction (at 152.4 46.99) (diameter 0) (color 0 0 0 0)
+  )
+  (junction (at 152.4 52.07) (diameter 0) (color 0 0 0 0)
+  )
   (junction (at 203.835 118.11) (diameter 0) (color 0 0 0 0)
   )
   (junction (at 40.005 37.465) (diameter 0) (color 0 0 0 0)
   )
+  (junction (at 151.765 34.29) (diameter 0) (color 0 0 0 0)
+  )
   (junction (at 170.815 42.545) (diameter 0) (color 0 0 0 0)
   )
@@
   (junction (at 145.415 95.885) (diameter 0) (color 0 0 0 0)
   )
+  (junction (at 152.4 49.53) (diameter 0) (color 0 0 0 0)
+  )
   (junction (at 220.345 79.375) (diameter 0) (color 0 0 0 0)
   )
@@
   (junction (at 186.69 89.535) (diameter 0) (color 0 0 0 0)
   )
+  (junction (at 151.765 36.83) (diameter 0) (color 0 0 0 0)
+  )
   (junction (at 170.815 47.625) (diameter 0) (color 0 0 0 0)
+  )
+  (junction (at 151.765 39.37) (diameter 0) (color 0 0 0 0)
   )
   (junction (at 220.345 76.835) (diameter 0) (color 0 0 0 0)
@@
   (no_connect (at 192.405 74.295))
   (no_connect (at 192.405 84.455))
-  (no_connect (at 192.405 86.995))
   (no_connect (at 215.265 71.755))
   (no_connect (at 192.405 81.915))
@@
     (stroke (width 0) (type default))
   )
+  (wire (pts (xy 152.4 52.07) (xy 152.4 49.53))
+    (stroke (width 0) (type default))
+  )
   (wire (pts (xy 170.815 47.625) (xy 170.815 49.53))
     (stroke (width 0) (type default))
@@
     (stroke (width 0) (type default))
   )
+  (wire (pts (xy 186.69 86.995) (xy 192.405 86.995))
+    (stroke (width 0) (type default))
+  )
   (wire (pts (xy 155.575 104.14) (xy 155.575 106.045))
     (stroke (width 0) (type default))
@@
     (stroke (width 0) (type default))
   )
+  (wire (pts (xy 151.765 36.83) (xy 151.765 34.29))
+    (stroke (width 0) (type default))
+  )
   (wire (pts (xy 67.945 83.185) (xy 98.425 83.185))
     (stroke (width 0) (type default))
   )
+  (wire (pts (xy 148.59 49.53) (xy 152.4 49.53))
+    (stroke (width 0) (type default))
+  )
   (wire (pts (xy 40.005 31.75) (xy 40.005 37.465))
     (stroke (width 0) (type default))
@@
     (stroke (width 0) (type default))
   )
+  (wire (pts (xy 148.59 52.07) (xy 152.4 52.07))
+    (stroke (width 0) (type default))
+  )
   (wire (pts (xy 192.405 69.215) (xy 186.69 69.215))
     (stroke (width 0) (type default))
@@
     (stroke (width 0) (type default))
   )
+  (wire (pts (xy 151.765 26.67) (xy 151.765 34.29))
+    (stroke (width 0) (type default))
+  )
   (wire (pts (xy 192.405 76.835) (xy 186.69 76.835))
     (stroke (width 0) (type default))
@@
     (stroke (width 0) (type default))
   )
+  (wire (pts (xy 186.69 86.995) (xy 186.69 89.535))
+    (stroke (width 0) (type default))
+  )
   (wire (pts (xy 67.945 73.025) (xy 67.945 76.2))
     (stroke (width 0) (type default))
@@
     (stroke (width 0) (type default))
   )
+  (wire (pts (xy 152.4 52.07) (xy 152.4 53.975))
+    (stroke (width 0) (type default))
+  )
+  (wire (pts (xy 148.59 29.21) (xy 160.655 29.21))
+    (stroke (width 0) (type default))
+  )
+  (wire (pts (xy 148.59 44.45) (xy 152.4 44.45))
+    (stroke (width 0) (type default))
+  )
+  (wire (pts (xy 148.59 36.83) (xy 151.765 36.83))
+    (stroke (width 0) (type default))
+  )
+  (wire (pts (xy 148.59 31.75) (xy 160.655 31.75))
+    (stroke (width 0) (type default))
+  )
   (wire (pts (xy 145.415 95.885) (xy 145.415 92.075))
     (stroke (width 0) (type default))
@@
     (stroke (width 0) (type default))
   )
+  (wire (pts (xy 148.59 34.29) (xy 151.765 34.29))
+    (stroke (width 0) (type default))
+  )
+  (wire (pts (xy 151.765 39.37) (xy 151.765 36.83))
+    (stroke (width 0) (type default))
+  )
   (wire (pts (xy 155.575 99.06) (xy 155.575 95.885))
     (stroke (width 0) (type default))
@@
     (stroke (width 0) (type default))
   )
+  (wire (pts (xy 148.59 41.91) (xy 151.765 41.91))
+    (stroke (width 0) (type default))
+  )
   (wire (pts (xy 200.66 118.11) (xy 203.835 118.11))
     (stroke (width 0) (type default))
   )
+  (wire (pts (xy 152.4 49.53) (xy 152.4 46.99))
+    (stroke (width 0) (type default))
+  )
   (wire (pts (xy 192.405 89.535) (xy 186.69 89.535))
     (stroke (width 0) (type default))
@@
     (stroke (width 0) (type default))
   )
+  (wire (pts (xy 152.4 46.99) (xy 152.4 44.45))
+    (stroke (width 0) (type default))
+  )
+  (wire (pts (xy 148.59 46.99) (xy 152.4 46.99))
+    (stroke (width 0) (type default))
+  )
   (wire (pts (xy 189.865 109.22) (xy 195.58 109.22))
     (stroke (width 0) (type default))
@@
     (stroke (width 0) (type default))
   )
+  (wire (pts (xy 151.765 41.91) (xy 151.765 39.37))
+    (stroke (width 0) (type default))
+  )
   (wire (pts (xy 60.96 37.465) (xy 60.96 41.275))
     (stroke (width 0) (type default))
@@
     (stroke (width 0) (type default))
   )
+  (wire (pts (xy 148.59 39.37) (xy 151.765 39.37))
+    (stroke (width 0) (type default))
+  )
   (wire (pts (xy 135.89 49.53) (xy 123.825 49.53))
     (stroke (width 0) (type default))
   )
-  (wire (pts (xy 186.69 79.375) (xy 186.69 89.535))
+  (wire (pts (xy 186.69 79.375) (xy 186.69 86.995))
     (stroke (width 0) (type default))
   )
@@
     (effects (font (size 1.27 1.27)) (justify left bottom))
   )
-  (label "SWCLK" (at 209.55 40.005 180) (fields_autoplaced)
+  (label "SWDCLK" (at 209.55 40.005 180) (fields_autoplaced)
+    (effects (font (size 1.27 1.27)) (justify right bottom))
+  )
+  (label "PB1" (at 160.655 31.75 180) (fields_autoplaced)
     (effects (font (size 1.27 1.27)) (justify right bottom))
   )
@@
     (effects (font (size 1.27 1.27)) (justify right bottom))
   )
+  (label "PB0" (at 160.655 29.21 180) (fields_autoplaced)
+    (effects (font (size 1.27 1.27)) (justify right bottom))
+  )
   (label "PA2" (at 123.825 34.29 0) (fields_autoplaced)
     (effects (font (size 1.27 1.27)) (justify left bottom))
@@
   (label "PA2" (at 86.36 95.885 0) (fields_autoplaced)
     (effects (font (size 1.27 1.27)) (justify left bottom))
+  )
+  (symbol (lib_id "power:VCC") (at 151.765 26.67 0) (mirror y) (unit 1)
+    (in_bom yes) (on_board yes) (dnp no)
+    (property "Reference" "#PWR017" (at 151.765 30.48 0)
+      (effects (font (size 1.27 1.27)) hide)
+    )
+    (property "Value" "VCC" (at 151.765 23.1681 0)
+      (effects (font (size 1.27 1.27)))
+    )
+    (property "Footprint" "" (at 151.765 26.67 0)
+      (effects (font (size 1.27 1.27)) hide)
+    )
+    (property "Datasheet" "" (at 151.765 26.67 0)
+      (effects (font (size 1.27 1.27)) hide)
+    )
+    (pin "1")
+    (instances
+      (project "PuyoPuya"
+        (path "/a56fab31-b869-4c40-8d6b-eff76b19676a"
+          (reference "#PWR017") (unit 1)
+        )
+      )
+    )
+  )
+  (symbol (lib_id "power:GND") (at 152.4 53.975 0) (unit 1)
+    (in_bom yes) (on_board yes) (dnp no) (fields_autoplaced)
+    (property "Reference" "#PWR016" (at 152.4 60.325 0)
+      (effects (font (size 1.27 1.27)) hide)
+    )
+    (property "Value" "GND" (at 152.4 58.1105 0)
+      (effects (font (size 1.27 1.27)))
+    )
+    (property "Footprint" "" (at 152.4 53.975 0)
+      (effects (font (size 1.27 1.27)) hide)
+    )
+    (property "Datasheet" "" (at 152.4 53.975 0)
+      (effects (font (size 1.27 1.27)) hide)
+    )
+    (pin "1")
+    (instances
+      (project "PuyoPuya"
+        (path "/a56fab31-b869-4c40-8d6b-eff76b19676a"
+          (reference "#PWR016") (unit 1)
+        )
+      )
+    )
   )
   (symbol (lib_id "Device:C_Small") (at 155.575 101.6 0) (unit 1)
@@
     )
   )
-  (symbol (lib_id "Connector_Generic:Conn_01x10") (at 140.97 39.37 0) (unit 1)
-    (in_bom yes) (on_board yes) (dnp no) (fields_autoplaced)
-    (property "Reference" "J1" (at 143.002 39.9963 0)
+  (symbol (lib_id "Connector_Generic:Conn_02x10_Odd_Even") (at 140.97 39.37 0) (unit 1)
+    (in_bom yes) (on_board yes) (dnp no)
+    (property "Reference" "J1" (at 140.97 23.495 0)
       (effects (font (size 1.27 1.27)) (justify left))
     )
-    (property "Value" "Conn_01x10" (at 143.002 41.9173 0)
+    (property "Value" "Conn_02x10" (at 136.525 25.416 0)
       (effects (font (size 1.27 1.27)) (justify left))
     )
-    (property "Footprint" "Connector_PinSocket_2.54mm:PinSocket_1x10_P2.54mm_Vertical" (at 140.97 39.37 0)
+    (property "Footprint" "Connector_PinSocket_2.54mm:PinSocket_2x10_P2.54mm_Vertical" (at 140.97 39.37 0)
       (effects (font (size 1.27 1.27)) hide)
     )
@@
     (pin "1")
     (pin "10")
+    (pin "11")
+    (pin "12")
+    (pin "13")
+    (pin "14")
+    (pin "15")
+    (pin "16")
+    (pin "17")
+    (pin "18")
+    (pin "19")
     (pin "2")
+    (pin "20")
     (pin "3")
     (pin "4")

Commit message: Fix routing
Parts:
- added C4: 1uF, Capacitor_SMD:C_0805_2012Metric_Pad1.18x1.45mm_HandSolder, symbol Device:C_Small
- added C5: 10uF, Capacitor_SMD:C_0805_2012Metric_Pad1.18x1.45mm_HandSolder, symbol Device:C_Small
Connections:
- net GND: now also C4.2, C5.2
- net VCC: now also C4.1, C5.1
Changed lines of the file:
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@@
+    )
+  )
+  (symbol (lib_id "power:GND") (at 165.735 72.39 0) (unit 1)
+    (in_bom yes) (on_board yes) (dnp no) (fields_autoplaced)
+    (property "Reference" "#PWR021" (at 165.735 78.74 0)
+      (effects (font (size 1.27 1.27)) hide)
+    )
+    (property "Value" "GND" (at 165.735 76.5255 0)
+      (effects (font (size 1.27 1.27)))
+    )
+    (property "Footprint" "" (at 165.735 72.39 0)
+      (effects (font (size 1.27 1.27)) hide)
+    )
+    (property "Datasheet" "" (at 165.735 72.39 0)
+      (effects (font (size 1.27 1.27)) hide)
+    )
+    (pin "1")
+    (instances
+      (project "PuyoPuya"
+        (path "/a56fab31-b869-4c40-8d6b-eff76b19676a"
+          (reference "#PWR021") (unit 1)
+        )
+      )
     )
   )
@@
         (path "/a56fab31-b869-4c40-8d6b-eff76b19676a"
           (reference "#PWR010") (unit 1)
+        )
+      )
+    )
+  )
+  (symbol (lib_id "power:VCC") (at 165.735 67.31 0) (unit 1)
+    (in_bom yes) (on_board yes) (dnp no) (fields_autoplaced)
+    (property "Reference" "#PWR018" (at 165.735 71.12 0)
+      (effects (font (size 1.27 1.27)) hide)
+    )
+    (property "Value" "VCC" (at 165.735 63.8081 0)
+      (effects (font (size 1.27 1.27)))
+    )
+    (property "Footprint" "" (at 165.735 67.31 0)
+      (effects (font (size 1.27 1.27)) hide)
+    )
+    (property "Datasheet" "" (at 165.735 67.31 0)
+      (effects (font (size 1.27 1.27)) hide)
+    )
+    (pin "1")
+    (instances
+      (project "PuyoPuya"
+        (path "/a56fab31-b869-4c40-8d6b-eff76b19676a"
+          (reference "#PWR018") (unit 1)
+        )
+      )
+    )
+  )
+  (symbol (lib_id "Device:C_Small") (at 175.895 69.85 0) (unit 1)
+    (in_bom yes) (on_board yes) (dnp no) (fields_autoplaced)
+    (property "Reference" "C5" (at 178.2191 69.2126 0)
+      (effects (font (size 1.27 1.27)) (justify left))
+    )
+    (property "Value" "10uF" (at 178.2191 71.1336 0)
+      (effects (font (size 1.27 1.27)) (justify left))
+    )
+    (property "Footprint" "Capacitor_SMD:C_0805_2012Metric_Pad1.18x1.45mm_HandSolder" (at 175.895 69.85 0)
+      (effects (font (size 1.27 1.27)) hide)
+    )
+    (property "Datasheet" "~" (at 175.895 69.85 0)
+      (effects (font (size 1.27 1.27)) hide)
+    )
+    (pin "1")
+    (pin "2")
+    (instances
+      (project "PuyoPuya"
+        (path "/a56fab31-b869-4c40-8d6b-eff76b19676a"
+          (reference "C5") (unit 1)
         )
       )
@@
     )
   )
+  (symbol (lib_id "Device:C_Small") (at 165.735 69.85 0) (unit 1)
+    (in_bom yes) (on_board yes) (dnp no) (fields_autoplaced)
+    (property "Reference" "C4" (at 168.0591 69.2126 0)
+      (effects (font (size 1.27 1.27)) (justify left))
+    )
+    (property "Value" "1uF" (at 168.0591 71.1336 0)
+      (effects (font (size 1.27 1.27)) (justify left))
+    )
+    (property "Footprint" "Capacitor_SMD:C_0805_2012Metric_Pad1.18x1.45mm_HandSolder" (at 165.735 69.85 0)
+      (effects (font (size 1.27 1.27)) hide)
+    )
+    (property "Datasheet" "~" (at 165.735 69.85 0)
+      (effects (font (size 1.27 1.27)) hide)
+    )
+    (pin "1")
+    (pin "2")
+    (instances
+      (project "PuyoPuya"
+        (path "/a56fab31-b869-4c40-8d6b-eff76b19676a"
+          (reference "C4") (unit 1)
+        )
+      )
+    )
+  )
   (symbol (lib_id "Device:LED") (at 186.055 118.11 0) (mirror y) (unit 1)
     (in_bom yes) (on_board yes) (dnp no) (fields_autoplaced)
@@
     )
   )
+  (symbol (lib_id "power:GND") (at 175.895 72.39 0) (unit 1)
+    (in_bom yes) (on_board yes) (dnp no) (fields_autoplaced)
+    (property "Reference" "#PWR020" (at 175.895 78.74 0)
+      (effects (font (size 1.27 1.27)) hide)
+    )
+    (property "Value" "GND" (at 175.895 76.5255 0)
+      (effects (font (size 1.27 1.27)))
+    )
+    (property "Footprint" "" (at 175.895 72.39 0)
+      (effects (font (size 1.27 1.27)) hide)
+    )
+    (property "Datasheet" "" (at 175.895 72.39 0)
+      (effects (font (size 1.27 1.27)) hide)
+    )
+    (pin "1")
+    (instances
+      (project "PuyoPuya"
+        (path "/a56fab31-b869-4c40-8d6b-eff76b19676a"
+          (reference "#PWR020") (unit 1)
+        )
+      )
+    )
+  )
   (symbol (lib_id "power:VCC") (at 145.415 92.075 0) (unit 1)
     (in_bom yes) (on_board yes) (dnp no) (fields_autoplaced)
@@
         )
       )
+    )
+  )
+  (symbol (lib_id "power:VCC") (at 175.895 67.31 0) (unit 1)
+    (in_bom yes) (on_board yes) (dnp no) (fields_autoplaced)
+    (property "Reference" "#PWR019" (at 175.895 71.12 0)
+      (effects (font (size 1.27 1.27)) hide)
+    )
+    (property "Value" "VCC" (at 175.895 63.8081 0)
+      (effects (font (size 1.27 1.27)))
+    )
+    (property "Footprint" "" (at 175.895 67.31 0)
+      (effects (font (size 1.27 1.27)) hide)
+    )
+    (property "Datasheet" "" (at 175.895 67.31 0)
+      (effects (font (size 1.27 1.27)) hide)
+    )
+    (pin "1")
+    (instances
+      (project "PuyoPuya"
+        (path "/a56fab31-b869-4c40-8d6b-eff76b19676a"
+          (reference "#PWR019") (unit 1)
+        )
+      )

Commit message: CH340C
Parts:
- added C6, C7, C9: 0.1uF, Capacitor_SMD:C_0805_2012Metric_Pad1.18x1.45mm_HandSolder, symbol Device:C_Small
- added C8: 100nF, Capacitor_SMD:C_0805_2012Metric_Pad1.18x1.45mm_HandSolder, symbol Device:C_Small
- added U2: CH340C, Package_SO:SOP-16_3.9x9.9mm_P1.27mm, symbol Puya:CH340C
- C4: value 1uF -> 0.1uF
Connections:
- net GND: now also C6.2, C7.1, C9.2, U2.1 (GND)
- net NRST: now also C8.2
- net PA13/SWDIO: now also U2.2 (TXD); no longer J1.19 (Pin_19)
- net VCC: now also J1.19 (Pin_19), C6.1, C9.1, U2.16 (VCC)
- net USB_D+: now reaches J3.A6 (Dp1)
- net USB_D+: now also J3.B6 (Dp2), U2.5 (UD+)
- net USB_D-: now reaches J3.A7 (Dn1)
- net USB_D-: now also J3.B7 (Dn2), U2.6 (UD-)
- net SWDCLK renamed PY_TXD
- net PY_TXD: now also U2.3 (RXD)
- new net: C8.1, U2.13 (DTR)
- new net: C7.2, U2.4 (V3)
- no-connect marks 10 -> 12

Commit message: PuyoPuy030
Parts:
- added D3, D4: LED, LED_SMD:LED_0805_2012Metric_Pad1.15x1.40mm_HandSolder, symbol Device:LED
- added D5: BAT54C, Package_TO_SOT_SMD:SOT-23, symbol Diode:BAT54C
- added J4: UART_EN, Connector_PinHeader_2.54mm:PinHeader_2x02_P2.54mm_Vertical, symbol Connector_Generic:Conn_02x02_Odd_Even
- added JP1: VBUS, Connector_PinHeader_2.54mm:PinHeader_1x02_P2.54mm_Vertical, symbol Jumper:Jumper_2_Open
- added R10, R7, R8, R9: 1K, Resistor_SMD:R_0805_2012Metric_Pad1.20x1.40mm_HandSolder, symbol Device:R_Small_US
Connections:
- net PA13/SWDIO: now also J4.2 (Pin_2); no longer U2.2 (TXD)
- net PY_TXD: now also J4.3 (Pin_3), R8.1; no longer J2.4 (Pin_4), R2.1, U1.4 (PF1-OSCOUT/PA14)
- net VCC: now also D5.3, JP1.2 (B), R10.2, R9.2; no longer J1.6 (Pin_6), J2.1 (Pin_1), J3.A4 (VBUS), J3.A9 (VBUS), J3.B4 (VBUS), J3.B9 (VBUS)
- new net: D3.2 (A), R9.1
- new net: D5.1, D5.2, J2.1 (Pin_1)
- new net: D4.1 (K), R8.2
- new net: J3.A4 (VBUS), J3.A9 (VBUS), J3.B4 (VBUS), J3.B9 (VBUS), JP1.1 (A)
- new net: D4.2 (A), R10.1
- new net: D3.1 (K), R7.2
- new net PA13: J1.6 (Pin_6)
- new net PY_RXD: J4.1 (Pin_1), R7.1, U2.2 (TXD)
- new net SWDCLK: J2.4 (Pin_4), J4.4 (Pin_4), R2.1, U1.4 (PF1-OSCOUT/PA14)
Other:
- moved on the sheet: R1, R2
