File: PuyoPuya/PuyoPuya.kicad_pcb (KiCad board)
At the start: 2 copper layers, 8.7 x 4.5 mm, 17 parts, among them J1 Conn_01x10, J2 SWD, J3 USB4085-GF-A, SW1 SW_Push, U1 PY32F003W16S6TU

Commit message: Boarb
Parts:
- J1: value Conn_01x10 -> Conn_02x10; footprint Connector_PinSocket_2.54mm:PinSocket_1x10_P2.54mm_Vertical -> Connector_PinSocket_2.54mm:PinSocket_2x10_P2.54mm_Vertical
- moved J1 36.0 mm to (156.7, 74.9), turned to 180 degrees
- moved TP1 33.9 mm to (149.4, 52.8)
- moved C2 32.2 mm to (146.5, 62.1), turned to 90 degrees
- moved C1 29.0 mm to (144.2, 62.1), turned to 90 degrees
- moved C3 20.4 mm to (133.9, 66.1), turned to -90 degrees
- moved SW1 16.5 mm to (135.1, 71.6), turned to -90 degrees
- moved R5 15.3 mm to (151.4, 69.8), turned to 90 degrees
- moved D1 14.0 mm to (148.3, 68.6), turned to 180 degrees
- moved R1 10.0 mm to (141.0, 61.7), turned to -90 degrees
- moved R3 9.38 mm to (136.1, 66.1), turned to 90 degrees
- moved D2 8.67 mm to (148.3, 66.3), turned to 180 degrees
- moved J3 7.78 mm to (125.3, 53.3), turned to -90 degrees
- moved U1 7.38 mm to (142.2, 69.5)
- moved R6 7.10 mm to (151.4, 64.5), turned to -90 degrees
- moved R2 6.46 mm to (138.0, 60.7)
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Connections:
- J1 pad 10: /PA13/SWDIO -> VCC
- J1 pad 2: /PA1 -> /PB0
- J1 pad 3: /PA2 -> /PA1
- J1 pad 4: /PA3 -> /PB1
- J1 pad 5: /PA4 -> /PA2
- J1 pad 6: /PA5 -> VCC
- J1 pad 7: /PA6 -> /PA3
- J1 pad 8: /PA7 -> VCC
- J1 pad 9: /PA12 -> /PA4
- J2 pad 4: /SWCLK -> /SWDCLK
- J3 pad B12: unconnected-(J3-GND-PadB12) -> GND
Routing:
- net /PA13/SWDIO: track 0.00 -> 44.2 mm, vias 0 -> 3
- net /NRST: track 0.00 -> 33.4 mm, vias 0 -> 1
- net /PB1: track 0.00 -> 25.5 mm, vias 0 -> 2
- net /PA0: track 0.00 -> 25.0 mm
- net /PB0: track 0.00 -> 24.9 mm, vias 0 -> 2
- net /PA1: track 0.00 -> 23.6 mm
- net /PA12: track 0.00 -> 23.4 mm, vias 0 -> 2
- net GND: track 0.00 -> 23.0 mm
- net /PA7: track 0.00 -> 21.4 mm, vias 0 -> 1
- net /PA2: track 0.00 -> 20.3 mm
- net /PA6: track 0.00 -> 19.5 mm, vias 0 -> 1
- net /SWDCLK: track 0.00 -> 19.0 mm, vias 0 -> 1
- net /PA5: track 0.00 -> 18.1 mm, vias 0 -> 1
- net /PA4: track 0.00 -> 16.5 mm, vias 0 -> 1
- net /PA3: track 0.00 -> 16.1 mm
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- added copper zone on F.Cu, net GND
- added copper zone on B.Cu, net VCC
Other:
- board size 8.7 x 4.5 mm -> 43.4 x 26.9 mm
- board text added: "PA0"
- board text added: "PA1"
- board text added: "PA12"
- board text added: "PA13"
- board text added: "PA2"
- board text added: "PA3"
- board text added: "PA4"
- board text added: "PA5"
- board text added: "PA6"
- board text added: "PA7"
- board text added: "PB0"
- board text added: "PB1"
- board text added: "POWER"
- board text added: "PY32F003"
- board text added: "RESET"
- board text added: "SWD"
- board text added: "TRACE"

Commit message: Fix routing
Parts:
- added C4: 1uF, Capacitor_SMD:C_0805_2012Metric_Pad1.18x1.45mm_HandSolder, F.Cu at (131.7, 59.2)
- added C5: 10uF, Capacitor_SMD:C_0805_2012Metric_Pad1.18x1.45mm_HandSolder, F.Cu at (128.7, 59.2)
Routing:
- net VCC: track 9.87 -> 67.7 mm
- net GND: track 23.0 -> 0.00 mm, vias 0 -> 8
- net /PB1: track 25.5 -> 20.3 mm, vias 2 -> 1
- net /PB0: track 24.9 -> 20.0 mm, vias 2 -> 1
- net /PA7: track 21.4 -> 26.2 mm, vias 1 -> 0
- net /PA6: track 19.5 -> 23.9 mm, vias 1 -> 0
- net /PA5: track 18.1 -> 21.6 mm, vias 1 -> 0
- net /PA4: track 16.5 -> 19.3 mm, vias 1 -> 0
- net Net-(D1-K): track 0.00 -> 2.13 mm
- net Net-(R4-Pad1): track 12.7 -> 14.7 mm, vias 2 -> 0
- net /PA12: track 23.4 -> 21.9 mm, vias 2 -> 0
- net /PA13/SWDIO: track 44.2 -> 43.0 mm, vias 3 -> 0
- net /PA0: track 25.0 -> 26.1 mm
- net /PA1: track 23.6 -> 24.6 mm
- net /PA3: track 16.1 -> 17.0 mm
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- added copper zone on B.Cu, net GND
- removed copper zone on B.Cu, net VCC
Other:
- board size 43.4 x 26.9 mm -> 45.4 x 27.3 mm
- board text added: "GND"
- board text added: "VCC"

Commit message: CH340C
Parts:
- added C6: 0.1uF, Capacitor_SMD:C_0805_2012Metric_Pad1.18x1.45mm_HandSolder, F.Cu at (126.8, 53.0)
- added C7: 0.1uF, Capacitor_SMD:C_0805_2012Metric_Pad1.18x1.45mm_HandSolder, F.Cu at (128.3, 62.9)
- added C8: 100nF, Capacitor_SMD:C_0805_2012Metric_Pad1.18x1.45mm_HandSolder, F.Cu at (129.6, 58.8)
- added C9: 0.1uF, Capacitor_SMD:C_0805_2012Metric_Pad1.18x1.45mm_HandSolder, F.Cu at (119.7, 50.4)
- added U2: CH340C, Package_SO:SOP-16_3.9x9.9mm_P1.27mm, F.Cu at (123.2, 59.4)
- C4: value 1uF -> 0.1uF
- moved C4 14.0 mm to (118.2, 63.0)
- moved C5 11.1 mm to (119.7, 52.7), turned to 0 degrees
- moved J3 9.09 mm to (116.3, 52.7)
- moved J2 3.18 mm to (133.4, 52.2)
- moved TP1 3.18 mm to (149.4, 49.7)
- turned C3 to 90 degrees
- turned R3 to -90 degrees
Connections:
- net /SWDCLK renamed /PY_TXD
- J1 pad 19: /PA13/SWDIO -> VCC
- J3 pad A6: unconnected-(J3-Dp1-PadA6) -> /USB_D+
- J3 pad A7: unconnected-(J3-Dn1-PadA7) -> /USB_D-
- J3 pad B6: unconnected-(J3-Dp2-PadB6) -> /USB_D+
- J3 pad B7: unconnected-(J3-Dn2-PadB7) -> /USB_D-
Routing:
- net VCC: track 67.7 -> 115.8 mm, vias 5 -> 0
- net /PY_TXD: track 18.9 -> 38.7 mm, vias 0 -> 4
- net Net-(U2-V3): track 0.00 -> 12.8 mm
- net /NRST: track 33.5 -> 45.9 mm
- net /USB_D-: track 0.00 -> 9.58 mm
- net /USB_D+: track 0.00 -> 9.51 mm
- net /PA13/SWDIO: track 43.0 -> 39.8 mm, vias 0 -> 2
- net Net-(U2-DTR): track 0.00 -> 2.85 mm
- net Net-(R4-Pad1): track 14.7 -> 12.1 mm, vias 0 -> 2
- net /PB1: track 20.3 -> 18.0 mm
- net /PA1: track 24.6 -> 22.8 mm
- net /PA0: track 26.1 -> 24.3 mm
- net /PB0: track 20.0 -> 18.5 mm
- net /PA12: track 21.9 -> 23.3 mm
- net /PA3: track 17.0 -> 17.7 mm
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Other:
- board size 45.4 x 27.3 mm -> 55.9 x 33.5 mm
- board text removed: "PA13"
- board text removed: "POWER"

Commit message: PuyoPuy030
Parts:
- added D3: LED, LED_SMD:LED_0805_2012Metric_Pad1.15x1.40mm_HandSolder, F.Cu at (147.1, 57.5)
- added D4: LED, LED_SMD:LED_0805_2012Metric_Pad1.15x1.40mm_HandSolder, F.Cu at (147.1, 55.4)
- added D5: BAT54C, Package_TO_SOT_SMD:SOT-23, F.Cu at (134.0, 56.4)
- added J4: UART_EN, Connector_PinHeader_2.54mm:PinHeader_2x02_P2.54mm_Vertical, F.Cu at (133.3, 60.4)
- added JP1: VBUS, Connector_PinHeader_2.54mm:PinHeader_1x02_P2.54mm_Vertical, F.Cu at (110.7, 63.1)
- added R10: 1K, Resistor_SMD:R_0805_2012Metric_Pad1.20x1.40mm_HandSolder, F.Cu at (147.8, 51.7)
- added R7: 1K, Resistor_SMD:R_0805_2012Metric_Pad1.20x1.40mm_HandSolder, F.Cu at (143.3, 57.5)
- added R8: 1K, Resistor_SMD:R_0805_2012Metric_Pad1.20x1.40mm_HandSolder, F.Cu at (143.3, 55.4)
- added R9: 1K, Resistor_SMD:R_0805_2012Metric_Pad1.20x1.40mm_HandSolder, F.Cu at (149.9, 51.7)
- added REF**: Mount_2.1, Puya:Mount_2.1, F.Cu at (162.1, 78.3)
- added REF**: Mount_2.1, Puya:Mount_2.1, F.Cu at (110.2, 78.3)
- added REF**: Mount_2.1, Puya:Mount_2.1, F.Cu at (162.1, 48.7)
- added REF**: Mount_2.1, Puya:Mount_2.1, F.Cu at (110.2, 48.7)
- moved TP1 20.4 mm to (129.0, 48.5)
- moved C8 3.03 mm to (126.7, 58.0), turned to -90 degrees
- moved D1 2.76 mm to (148.1, 71.3)
- moved D2 2.76 mm to (148.1, 69.0)
- moved R3 2.76 mm to (135.9, 68.8)
- moved U1 2.76 mm to (141.9, 72.2)
- moved C3 2.76 mm to (133.6, 68.8)
- moved R1 2.76 mm to (140.7, 64.5)
- moved R2 2.76 mm to (137.7, 63.5)
- moved R5 2.76 mm to (151.1, 72.6)
- moved R6 2.76 mm to (151.1, 67.3)
- moved SW1 2.76 mm to (134.8, 74.4)
- moved C1 2.76 mm to (143.9, 64.8)
- moved C2 2.76 mm to (146.2, 64.8)
- moved R4 2.76 mm to (137.7, 65.8)
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Connections:
- J1 pad 6: VCC -> /PA13
- J2 pad 1: VCC -> Net-(J2-Pin_1)
- J2 pad 4: /PY_TXD -> /SWDCLK
- J3 pad A4: VCC -> Net-(JP1-A)
- J3 pad A9: VCC -> Net-(JP1-A)
- J3 pad B4: VCC -> Net-(JP1-A)
- J3 pad B9: VCC -> Net-(JP1-A)
- R2 pad 1: /PY_TXD -> /SWDCLK
- U1 pad 4: /PY_TXD -> /SWDCLK
- U2 pad 2: /PA13/SWDIO -> /PY_RXD
Routing:
- net VCC: track 115.8 -> 157.9 mm
- net /SWDCLK: track 0.00 -> 35.8 mm, vias 0 -> 1
- net /PY_RXD: track 0.00 -> 26.5 mm, vias 0 -> 2
- net Net-(JP1-A): track 0.00 -> 15.5 mm
- net /PY_TXD: track 38.7 -> 28.2 mm, vias 4 -> 2
- net /PA13/SWDIO: track 39.8 -> 31.7 mm, vias 2 -> 1
- net Net-(D3-A): track 0.00 -> 5.53 mm
- net Net-(J2-Pin_1): track 0.00 -> 5.27 mm
- net /NRST: track 45.9 -> 50.9 mm, vias 1 -> 5
- net /PA2: track 20.3 -> 23.4 mm
- net /PA4: track 19.2 -> 22.2 mm
- net /PA5: track 21.6 -> 24.6 mm
- net /PA6: track 23.9 -> 26.7 mm
- net Net-(D4-A): track 0.00 -> 2.77 mm
- net Net-(U2-V3): track 12.8 -> 10.4 mm
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Other:
- outline, holes or cut-outs redrawn
- board text added: "CK"
- board text added: "IO"
- board text added: "JLCJLCJLCJLC"
- board text added: "PA13"
- board text added: "RST"
- board text added: "RX"
- board text added: "SWO"
- board text added: "TX"
- board text added: "UART En"
- board text added: "VBUS"
- board text added: "rev. 1 github.com/kvanderlaag"
